File: Hardware/TT7B v1.0.sch (EAGLE design)
At the start: 74 parts, among them U1 SAML21E18B-MUT, U10 W3011A, U11 SI5351B, U12 TPS3839, U13 MIC9407, U14 SIT1552, U15 VEML6030, U16 TPS61099, U17 TPS61099, U2 UBLOX_ZOE-M8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

Commit message: Add files via upload
Parts:
- R15: value 0Ω -> 0R
- R21: value 1MΩ -> 1M
- R4: value 1kΩ -> 1k
Changed lines of the file:
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@@
 <part name="SUPPLY25" library="supply2" deviceset="GND" device=""/>
 <part name="C10" library="TT7" deviceset="CAP0402" device="" value="18nF"/>
-<part name="R4" library="TT7" deviceset="RES0402" device="" value="1kΩ"/>
+<part name="R4" library="TT7" deviceset="RES0402" device="" value="1k"/>
 <part name="SUPPLY26" library="supply2" deviceset="GND" device=""/>
 <part name="SUPPLY27" library="supply2" deviceset="GND" device=""/>
@@
 <part name="C16" library="TT7" deviceset="CAP0402" device="" value="100nF"/>
 <part name="SUPPLY43" library="supply2" deviceset="GND" device=""/>
-<part name="R15" library="TT7" deviceset="RES0402-3" device="" value="0Ω"/>
+<part name="R15" library="TT7" deviceset="RES0402-3" device="" value="0R"/>
 <part name="C17" library="TT7" deviceset="CAP0402" device="" value="100nF"/>
 <part name="C18" library="TT7" deviceset="CAP0402" device="" value="100nF"/>
@@
 <part name="D1" library="TT7" deviceset="ESD9R" device=""/>
 <part name="SUPPLY54" library="supply2" deviceset="GND" device=""/>
-<part name="R21" library="TT7" deviceset="RES0402" device="" value="1MΩ"/>
+<part name="R21" library="TT7" deviceset="RES0402" device="" value="1M"/>
 <part name="SUPPLY42" library="supply2" deviceset="GND" device=""/>
 <part name="U12" library="TT7" deviceset="TPS3839" device=""/>
